File: Hive PCB v0.1/Hive PCB v0.1.kicad_pcb (KiCad board)
At the start: 2 copper layers, 83.8 x 83.8 mm, 41 parts, among them J1 USB_B_Micro, Q1 BSS138

Commit message: Preliminary Place and Route on Hive PCV v0.1 Completed
Parts:
- JP2: value MCU_VUSB_SolderJumper -> VUSB_SolderJumper; footprint Jumper:SolderJumper-2_P1.3mm_Open_Pad1.0x1.5mm -> Jumper:SolderJumper-3_P1.3mm_Open_Pad1.0x1.5mm_NumberLabels
- moved R2 1.27 mm to (167.6, 94.0)
Connections:
- C1 pad 1: Net-(C1-Pad1) -> GND
- JP2 pad 1: VUSB -> Net-(Arduino_Nano_33_IoT1-Pad12)
- JP2 pad 2: Net-(Arduino_Nano_33_IoT1-Pad15) -> VUSB
Routing:
- net VUSB: track 0.00 -> 361.0 mm
- net GND: track 0.00 -> 132.9 mm, vias 0 -> 18
- net +3V3: track 0.00 -> 105.0 mm
- net LED_DATA_H: track 0.00 -> 55.9 mm, vias 0 -> 3
- net SCK: track 0.00 -> 52.2 mm, vias 0 -> 2
- net Net-(Arduino_Nano_33_IoT1-Pad15): track 0.00 -> 42.8 mm
- net IRQ_DWM1000: track 0.00 -> 40.0 mm, vias 0 -> 2
- net MISO: track 0.00 -> 35.7 mm, vias 0 -> 2
- net Net-(D11-Pad2): track 0.00 -> 33.7 mm, vias 0 -> 2
- net MOSI: track 0.00 -> 32.6 mm, vias 0 -> 2
- net LED_DATA_L: track 0.00 -> 32.4 mm
- net RSTn_DWM1000: track 0.00 -> 29.7 mm, vias 0 -> 2
- net CS_DWM1000: track 0.00 -> 29.6 mm, vias 0 -> 2
- net Net-(D10-Pad2): track 0.00 -> 28.7 mm
- net Net-(D10-Pad4): track 0.00 -> 28.6 mm, vias 0 -> 2
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- added copper zone on F.Cu, net GND
