File: Hive PCB v0.1/Hive PCB v0.1.1.kicad_pcb (KiCad board)
At the start: 2 copper layers, 83.8 x 83.8 mm, 41 parts, among them J1 USB_B_Micro, Q1 BSS138

Commit message: Corrected Solder Pads on Hive PCB 0.1
Removed solder mask from footprint of Arduino on PCB Version 0.1.
Other:
- board text added: "Designed by Mitchell Wu 2022.01.25 Last Updated 2022.02.28"
- board text added: "Hive PCB v0.1.1"
- board text removed: "Designed by Mitchell Wu 2022.01.25"
- board text removed: "Hive PCB v0.1"
Changed lines of the file:
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@@
     (pad "" np_thru_hole circle locked (at -20.73 -7.62) (size 1.651 1.651) (drill 1.651) (layers *.Cu *.Mask))
     (pad "" np_thru_hole circle locked (at 19.91 7.62) (size 1.651 1.651) (drill 1.651) (layers *.Cu *.Mask))
-    (pad "1" smd rect locked (at -18.19 9.1) (size 1.56 2) (layers "F.Cu" "F.Paste")
+    (pad "1" smd rect locked (at -18.19 9.1) (size 1.56 2) (layers "F.Cu" "F.Paste" "F.Mask")
       (net 1 "SCK"))
-    (pad "2" smd rect locked (at -15.65 9.1) (size 1.56 2) (layers "F.Cu" "F.Paste")
+    (pad "2" smd rect locked (at -15.65 9.1) (size 1.56 2) (layers "F.Cu" "F.Paste" "F.Mask")
       (net 2 "Net-(Arduino_Nano_33_IoT1-Pad2)"))
-    (pad "3" smd rect locked (at -13.11 9.1) (size 1.56 2) (layers "F.Cu" "F.Paste")
+    (pad "3" smd rect locked (at -13.11 9.1) (size 1.56 2) (layers "F.Cu" "F.Paste" "F.Mask")
       (net 3 "Net-(Arduino_Nano_33_IoT1-Pad3)"))
-    (pad "4" smd rect locked (at -10.57 9.1) (size 1.56 2) (layers "F.Cu" "F.Paste")
+    (pad "4" smd rect locked (at -10.57 9.1) (size 1.56 2) (layers "F.Cu" "F.Paste" "F.Mask")
       (net 4 "Net-(Arduino_Nano_33_IoT1-Pad4)"))
-    (pad "5" smd rect locked (at -8.03 9.1) (size 1.56 2) (layers "F.Cu" "F.Paste")
+    (pad "5" smd rect locked (at -8.03 9.1) (size 1.56 2) (layers "F.Cu" "F.Paste" "F.Mask")
       (net 5 "Net-(Arduino_Nano_33_IoT1-Pad5)"))
-    (pad "6" smd rect locked (at -5.49 9.1) (size 1.56 2) (layers "F.Cu" "F.Paste")
+    (pad "6" smd rect locked (at -5.49 9.1) (size 1.56 2) (layers "F.Cu" "F.Paste" "F.Mask")
       (net 6 "Net-(Arduino_Nano_33_IoT1-Pad6)"))
-    (pad "7" smd rect locked (at -2.95 9.1) (size 1.56 2) (layers "F.Cu" "F.Paste")
+    (pad "7" smd rect locked (at -2.95 9.1) (size 1.56 2) (layers "F.Cu" "F.Paste" "F.Mask")
       (net 7 "Net-(Arduino_Nano_33_IoT1-Pad7)"))
-    (pad "8" smd rect locked (at -0.41 9.1) (size 1.56 2) (layers "F.Cu" "F.Paste")
+    (pad "8" smd rect locked (at -0.41 9.1) (size 1.56 2) (layers "F.Cu" "F.Paste" "F.Mask")
       (net 8 "Net-(Arduino_Nano_33_IoT1-Pad8)"))
-    (pad "9" smd rect locked (at 2.13 9.1) (size 1.56 2) (layers "F.Cu" "F.Paste")
+    (pad "9" smd rect locked (at 2.13 9.1) (size 1.56 2) (layers "F.Cu" "F.Paste" "F.Mask")
       (net 9 "Net-(Arduino_Nano_33_IoT1-Pad9)"))
-    (pad "10" smd rect locked (at 4.67 9.1) (size 1.56 2) (layers "F.Cu" "F.Paste")
+    (pad "10" smd rect locked (at 4.67 9.1) (size 1.56 2) (layers "F.Cu" "F.Paste" "F.Mask")
       (net 10 "Net-(Arduino_Nano_33_IoT1-Pad10)"))
-    (pad "11" smd rect locked (at 7.21 9.1) (size 1.56 2) (layers "F.Cu" "F.Paste")
+    (pad "11" smd rect locked (at 7.21 9.1) (size 1.56 2) (layers "F.Cu" "F.Paste" "F.Mask")
       (net 11 "Net-(Arduino_Nano_33_IoT1-Pad11)"))
-    (pad "12" smd rect locked (at 9.75 9.1) (size 1.56 2) (layers "F.Cu" "F.Paste")
+    (pad "12" smd rect locked (at 9.75 9.1) (size 1.56 2) (layers "F.Cu" "F.Paste" "F.Mask")
       (net 12 "Net-(Arduino_Nano_33_IoT1-Pad12)"))
-    (pad "13" smd rect locked (at 12.29 9.1) (size 1.56 2) (layers "F.Cu" "F.Paste")
+    (pad "13" smd rect locked (at 12.29 9.1) (size 1.56 2) (property pad_prop_bga) (layers "F.Cu" "F.Paste" "F.Mask")
       (net 13 "Net-(Arduino_Nano_33_IoT1-Pad13)"))
-    (pad "14" smd rect locked (at 14.83 9.1) (size 1.56 2) (layers "F.Cu" "F.Paste")
-      (net 14 "GND"))
-    (pad "15" smd rect locked (at 17.37 9.1) (size 1.56 2) (layers "F.Cu" "F.Paste")
+    (pad "14" smd rect locked (at 14.83 9.1) (size 1.56 2) (layers "F.Cu" "F.Paste" "F.Mask")
+      (net 14 "GND"))
+    (pad "15" smd rect locked (at 17.37 9.1) (size 1.56 2) (layers "F.Cu" "F.Paste" "F.Mask")
       (net 15 "Net-(Arduino_Nano_33_IoT1-Pad15)"))
-    (pad "16" smd rect locked (at 17.37 -9.1 180) (size 1.56 2) (layers "F.Cu" "F.Paste")
+    (pad "16" smd rect locked (at 17.37 -9.1 180) (size 1.56 2) (layers "F.Cu" "F.Paste" "F.Mask")
       (net 16 "Net-(Arduino_Nano_33_IoT1-Pad16)"))
-    (pad "17" smd rect locked (at 14.83 -9.1 180) (size 1.56 2) (layers "F.Cu" "F.Paste")
+    (pad "17" smd rect locked (at 14.83 -9.1 180) (size 1.56 2) (layers "F.Cu" "F.Paste" "F.Mask")
       (net 17 "Net-(Arduino_Nano_33_IoT1-Pad17)"))
-    (pad "18" smd rect locked (at 12.29 -9.1 180) (size 1.56 2) (layers "F.Cu" "F.Paste")
+    (pad "18" smd rect locked (at 12.29 -9.1 180) (size 1.56 2) (layers "F.Cu" "F.Paste" "F.Mask")
       (net 13 "Net-(Arduino_Nano_33_IoT1-Pad13)"))
-    (pad "19" smd rect locked (at 9.75 -9.1 180) (size 1.56 2) (layers "F.Cu" "F.Paste")
-      (net 14 "GND"))
-    (pad "20" smd rect locked (at 7.21 -9.1 180) (size 1.56 2) (layers "F.Cu" "F.Paste")
+    (pad "19" smd rect locked (at 9.75 -9.1 180) (size 1.56 2) (layers "F.Cu" "F.Paste" "F.Mask")
+      (net 14 "GND"))
+    (pad "20" smd rect locked (at 7.21 -9.1 180) (size 1.56 2) (layers "F.Cu" "F.Paste" "F.Mask")
       (net 18 "LED_DATA_L"))
-    (pad "21" smd rect locked (at 4.67 -9.1 180) (size 1.56 2) (layers "F.Cu" "F.Paste")
+    (pad "21" smd rect locked (at 4.67 -9.1 180) (size 1.56 2) (layers "F.Cu" "F.Paste" "F.Mask")
       (net 19 "Net-(Arduino_Nano_33_IoT1-Pad21)"))
-    (pad "22" smd rect locked (at 2.13 -9.1 180) (size 1.56 2) (layers "F.Cu" "F.Paste")
+    (pad "22" smd rect locked (at 2.13 -9.1 180) (size 1.56 2) (layers "F.Cu" "F.Paste" "F.Mask")
       (net 20 "Net-(Arduino_Nano_33_IoT1-Pad22)"))
-    (pad "23" smd rect locked (at -0.41 -9.1 180) (size 1.56 2) (layers "F.Cu" "F.Paste")
+    (pad "23" smd rect locked (at -0.41 -9.1 180) (size 1.56 2) (layers "F.Cu" "F.Paste" "F.Mask")
       (net 21 "Net-(Arduino_Nano_33_IoT1-Pad23)"))
-    (pad "24" smd rect locked (at -2.95 -9.1 180) (size 1.56 2) (layers "F.Cu" "F.Paste")
+    (pad "24" smd rect locked (at -2.95 -9.1 180) (size 1.56 2) (layers "F.Cu" "F.Paste" "F.Mask")
       (net 22 "Net-(Arduino_Nano_33_IoT1-Pad24)"))
-    (pad "25" smd rect locked (at -5.49 -9.1 180) (size 1.56 2) (layers "F.Cu" "F.Paste")
+    (pad "25" smd rect locked (at -5.49 -9.1 180) (size 1.56 2) (layers "F.Cu" "F.Paste" "F.Mask")
       (net 23 "Net-(Arduino_Nano_33_IoT1-Pad25)"))
-    (pad "26" smd rect locked (at -8.03 -9.1 180) (size 1.56 2) (layers "F.Cu" "F.Paste")
+    (pad "26" smd rect locked (at -8.03 -9.1 180) (size 1.56 2) (layers "F.Cu" "F.Paste" "F.Mask")
       (net 24 "IRQ_DWM1000"))
-    (pad "27" smd rect locked (at -10.57 -9.1 180) (size 1.56 2) (layers "F.Cu" "F.Paste")
+    (pad "27" smd rect locked (at -10.57 -9.1 180) (size 1.56 2) (layers "F.Cu" "F.Paste" "F.Mask")
       (net 25 "RSTn_DWM1000"))
-    (pad "28" smd rect locked (at -13.11 -9.1 180) (size 1.56 2) (layers "F.Cu" "F.Paste")
+    (pad "28" smd rect locked (at -13.11 -9.1 180) (size 1.56 2) (layers "F.Cu" "F.Paste" "F.Mask")
       (net 26 "CS_DWM1000"))
-    (pad "29" smd rect locked (at -15.65 -9.1 180) (size 1.56 2) (layers "F.Cu" "F.Paste")
+    (pad "29" smd rect locked (at -15.65 -9.1 180) (size 1.56 2) (layers "F.Cu" "F.Paste" "F.Mask")
       (net 27 "MOSI"))
-    (pad "30" smd rect locked (at -18.19 -9.1 180) (size 1.56 2) (layers "F.Cu" "F.Paste")
+    (pad "30" smd rect locked (at -18.19 -9.1 180) (size 1.56 2) (layers "F.Cu" "F.Paste" "F.Mask")
       (net 28 "MISO"))
   )
@@
   (gr_line (start 130.81 73.66) (end 130.81 85.09) (layer "Edge.Cuts") (width 0.15))
   (gr_circle (center 139.7 101.6) (end 181.61 101.6) (layer "Edge.Cuts") (width 0.15) (fill none))
-  (gr_text "Designed by Mitchell Wu\n2022.01.25" (at 139.7 130.81) (layer "B.SilkS")
+  (gr_text "Designed by Mitchell Wu\n2022.01.25\nLast Updated 2022.02.28" (at 139.7 130.81) (layer "B.SilkS")
     (effects (font (size 1 1) (thickness 0.15)) (justify mirror))
   )
@@
     (effects (font (size 1 1) (thickness 0.15)))
   )
-  (gr_text "Hive PCB v0.1" (at 118.11 85.09) (layer "F.SilkS")
+  (gr_text "Hive PCB v0.1.1" (at 118.11 85.09) (layer "F.SilkS")
     (effects (font (size 1.778 1.778) (thickness 0.254)))
   )
