File: Hive Bulb PCB v0.2/Hive Bulb PCB v0.2.sch (KiCad schematic (older format))
At the start: 39 parts, among them J1 USB_B_Micro, J2 Conn_01x02, J3 Conn_02x18_Odd_Even, J4 Conn_02x18_Odd_Even, U1 NCP1117-3.3_SOT223, U2 W25Q128JVS, U3 RP2040, Y1 ABLS-12.000MHZ-B4-T

Commit message: Updates to power delivery circuitry schema in Hive Lamp PCB v0.2.
Parts:
- added C? (x7): C, symbol Device:C
- added D?: D_Zener, symbol Device:D_Zener
- added F?: Fuse, symbol Device:Fuse
- added L? (x2): L, symbol Device:L
- added R? (x2): R_US, symbol Device:R_US
Connections:
- net GND: now also PS?.5 (-VO), C?.1, C?.2, C?.2, C?.2, D?.2 (A), R?.2
- net VBUS: now also C?.1, C?.1, D?.1 (K), L?.2, R?.1
- net at PS?.1 (AC(L)): now also L?.2
- net at PS?.2 (AC(N)): now also C?.2
- net at PS?.3 (+V(CAP)): now also C?.1
- net at PS?.4 (-V(CAP)): now also C?.2, C?.2
- net at PS?.6 (+VO): now also C?.1, L?.1
- new net: F?.1, R?.1
- new net: C?.1, L?.1, R?.2
- new net: C?.1, C?.2
Other:
- moved on the sheet: C1, C10, C11, C12, C13, C14, C15, C16, C17, C2, C3, C4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

Commit message: Completed BOM, Most of Schematic, Beginning Layout of Hive Bulb PCB v0.2.
Parts:
- removed C5: 100n, Capacitor_SMD:C_0402_1005Metric, symbol Device:C
- removed C? (x3): C, symbol Device:C
- removed J1: USB_B_Micro, RP2040_minimal:USB_Micro-B_Amphenol_10103594-0001LF_Horizontal_modified, symbol Connector:USB_B_Micro
- removed J3, J4: Conn_02x18_Odd_Even, Connector_PinHeader_2.54mm:PinHeader_2x18_P2.54mm_Vertical, symbol Connector_Generic:Conn_02x18_Odd_Even
- removed R1: 1k, Capacitor_SMD:C_0402_1005Metric, symbol Device:R
- removed R2: DNF, Capacitor_SMD:C_0402_1005Metric, symbol Device:R
- removed R?: R_US, symbol Device:R_US
- removed U2: W25Q128JVS, Package_SO:SOIC-8_5.23x5.23mm_P1.27mm, symbol Memory_Flash:W25Q128JVS
- added C19: 100nF, Capacitor_SMD:C_0805_2012Metric_Pad1.18x1.45mm_HandSolder, symbol Device:C
- added P_C1: 22uF, Capacitor_THT:CP_Radial_D12.5mm_P7.50mm, symbol Device:CP1
- added P_C2: 470uF, Capacitor_THT:CP_Radial_D8.0mm_P5.00mm, symbol Device:CP1
- added P_C3: 100uF, Capacitor_THT:CP_Radial_D6.3mm_P2.50mm, symbol Device:CP1
- added R4: 1k, Resistor_SMD:R_0805_2012Metric_Pad1.20x1.40mm_HandSolder, symbol Device:R
- added R5: DNF, Resistor_SMD:R_0805_2012Metric_Pad1.20x1.40mm_HandSolder, symbol Device:R
- added U2: W25Q40CLSNIG, W25Q40CLSNIG:SOIC127P600X175-8N, symbol W25Q40CLSNIG:W25Q40CLSNIG
- C10: renamed from C12; value 100n -> 100nF; footprint Capacitor_SMD:C_0402_1005Metric -> Capacitor_SMD:C_0805_2012Metric_Pad1.18x1.45mm_HandSolder
- C11: renamed from C13; value 100n -> 100nF; footprint Capacitor_SMD:C_0402_1005Metric -> Capacitor_SMD:C_0805_2012Metric_Pad1.18x1.45mm_HandSolder
- C12: renamed from C14; value 100n -> 100nF; footprint Capacitor_SMD:C_0402_1005Metric -> Capacitor_SMD:C_0805_2012Metric_Pad1.18x1.45mm_HandSolder
- C13: renamed from C15; value 100n -> 100nF; footprint Capacitor_SMD:C_0402_1005Metric -> Capacitor_SMD:C_0805_2012Metric_Pad1.18x1.45mm_HandSolder
- C14: renamed from C16; value 100n -> 100nF; footprint Capacitor_SMD:C_0402_1005Metric -> Capacitor_SMD:C_0805_2012Metric_Pad1.18x1.45mm_HandSolder
- C15: renamed from C6; value 100n -> 100nF; footprint Capacitor_SMD:C_0402_1005Metric -> Capacitor_SMD:C_0805_2012Metric_Pad1.18x1.45mm_HandSolder
- C16: renamed from C7; value 100n -> 100nF; footprint Capacitor_SMD:C_0402_1005Metric -> Capacitor_SMD:C_0805_2012Metric_Pad1.18x1.45mm_HandSolder
- C17: renamed from C8; value 1u -> 1uF; footprint Capacitor_SMD:C_0402_1005Metric -> Capacitor_SMD:C_0805_2012Metric_Pad1.18x1.45mm_HandSolder
- C18: renamed from C10; value 1u -> 1uF; footprint Capacitor_SMD:C_0402_1005Metric -> Capacitor_SMD:C_0805_2012Metric_Pad1.18x1.45mm_HandSolder
- C20: renamed from C2; value 27p -> 27pF; footprint Capacitor_SMD:C_0402_1005Metric -> Capacitor_SMD:C_0805_2012Metric_Pad1.18x1.45mm_HandSolder
- C21: renamed from C3; value 27p -> 27pF; footprint Capacitor_SMD:C_0402_1005Metric -> Capacitor_SMD:C_0805_2012Metric_Pad1.18x1.45mm_HandSolder
- C22: renamed from C17; value 10u -> 10uF; footprint Capacitor_SMD:C_0805_2012Metric -> Capacitor_SMD:C_0805_2012Metric_Pad1.18x1.45mm_HandSolder
- C6: renamed from C1; value 10u -> 10uF; footprint Capacitor_SMD:C_0805_2012Metric -> Capacitor_SMD:C_0805_2012Metric_Pad1.18x1.45mm_HandSolder
- C7: renamed from C4; value 10u -> 10uF; footprint Capacitor_SMD:C_0805_2012Metric -> Capacitor_SMD:C_0805_2012Metric_Pad1.18x1.45mm_HandSolder
- C8: renamed from C9; value 100n -> 100nF; footprint Capacitor_SMD:C_0402_1005Metric -> Capacitor_SMD:C_0805_2012Metric_Pad1.18x1.45mm_HandSolder
- C9: renamed from C11; value 100n -> 100nF; footprint Capacitor_SMD:C_0402_1005Metric -> Capacitor_SMD:C_0805_2012Metric_Pad1.18x1.45mm_HandSolder
- FUSE: renamed from F?; value Fuse -> 1A/300V
- J1: footprint Connector_USB:USB_Micro-B_GCT_USB3076-30-A -> USB3140-30-0140-1-C:GCT_USB3140-30-0140-1-C_REVE3
- LDM: renamed from L?; value L -> 1.2mH; footprint (none) -> Inductor_SMD:L_12x12mm_H8mm
- PS1: renamed from PS?; footprint CONV_LS05-13B05R3 -> LS05-13B05R3:CONV_LS05-13B05R3
- P_C4: renamed from C?; value C -> 100nF; footprint (none) -> Capacitor_SMD:C_0805_2012Metric_Pad1.18x1.45mm_HandSolder
- P_CX: renamed from C?; value C -> 100nF; footprint (none) -> Capacitor_SMD:C_1210_3225Metric_Pad1.33x2.70mm_HandSolder
- P_CY1, P_CY2: renamed from C?; value C -> 2.2nF; footprint (none) -> Capacitor_SMD:C_0805_2012Metric_Pad1.18x1.45mm_HandSolder
- P_L1: renamed from L?; value L -> 4.7uH
- P_R1: renamed from R?; value R_US -> 12
- R2: renamed from R3; footprint Capacitor_SMD:C_0402_1005Metric -> Resistor_SMD:R_0805_2012Metric_Pad1.20x1.40mm_HandSolder
- R3: renamed from R4; footprint Capacitor_SMD:C_0402_1005Metric -> Resistor_SMD:R_0805_2012Metric_Pad1.20x1.40mm_HandSolder
- R5: footprint Capacitor_SMD:C_0402_1005Metric -> Resistor_SMD:R_0805_2012Metric_Pad1.20x1.40mm_HandSolder
- TVS: renamed from D?; value D_Zener -> SMBJ7.0A; footprint (none) -> Diode_SMD:D_SMB_Handsoldering
- U3: footprint RP2040_minimal:RP2040-QFN-56 -> RP2040:RP2040-QFN-56
- Y1: footprint RP2040_minimal:Crystal_SMD_HC49-US -> RP2040:Crystal_SMD_HC49-US
- renumbered C16 to C5, R1 to R6
Connections:
- wire segments 354 -> 241
Other:
- note added: "Make sure C18 is close to pin 44 of RP2040"
- note removed: "Make sure C10 is close to pin 44 of RP2040"
- moved on the sheet: C22, C5, J1, R6, UWB_Module1

Commit message: Finished majority of component placement of Hive Bulb PCB v0.2.
Routing traces to come next.  Schematic still needs to be lightly adjusted.
Parts:
- removed H1, H2, H3, H4: MountingHole, MountingHole:MountingHole_2.7mm_M2.5, symbol Mechanical:MountingHole
- removed P_R1: 12, symbol Device:R_US
- added P_R1: SMW312RJT, SMW312RJT:RESM12055X530N, symbol SMW312RJT:SMW312RJT
- FUSE1: renamed from FUSE; footprint (none) -> Fuse:Fuse_2512_6332Metric_Pad1.52x3.35mm_HandSolder
- P_C1: value 22uF -> 10uF; footprint Capacitor_THT:CP_Radial_D12.5mm_P7.50mm -> Capacitor_SMD:CP_Elec_10x14.3
- P_L1: footprint (none) -> Inductor_SMD:L_Bourns-SRN4018
- R1: renamed from R4; value 1k -> 1K
- R2: renamed from R5; value 1k -> 10K
- R3: renamed from R5; value DNF -> 10K
- renumbered C20 to C1, C8 to C10, C18 to C11, C9 to C12, C10 to C13, C11 to C14, C12 to C15, C13 to C16, C14 to C17, C22 to C18, C21 to C2, C5 to C3, C6 to C4, C7 to C5, C19 to C6, C15 to C7, C16 to C8, C17 to C9, J2 to J1, J1 to J2, LDM to LDM1, P_CX to P_CX1, R2 to R4, R3 to R5, TVS to TVS1
Connections:
- wire segments 241 -> 234
Other:
- note added: "Make sure C11 is close to pin 44 of RP2040"
- note added: "Make sure C9 is close to pin 45 of RP2040"
- note removed: "Make sure C18 is close to pin 44 of RP2040"
- note removed: "Make sure C8 is close to pin 45 of RP2040"
- moved on the sheet: C18, FUSE1

Commit message: Revised power delivery and LED I/O for Hive Bulb PCB v0.2.
Parts:
- added D? (x4): LED, symbol Device:LED
- added D?: D_Schottky, symbol Device:D_Schottky
- added J?: Conn_01x03, symbol Connector_Generic:Conn_01x03
- added Q?: BSS138, Package_TO_SOT_SMD:SOT-23, symbol Transistor_FET:BSS138
- added Q?: DMG2305UX-7, SOT91P240X110-3N_DMG2305UX-7, symbol DMG2305UX-7:DMG2305UX-7
- added R? (x4): 330, Resistor_SMD:R_0805_2012Metric_Pad1.20x1.40mm_HandSolder, symbol Device:R_US
- added R? (x3): 10K, Resistor_SMD:R_0805_2012Metric_Pad1.20x1.40mm_HandSolder, symbol Device:R_US
Connections:
- net +3V3: now also Q?.1 (G), R?.1
- net GND: now also D?.1 (K), D?.1 (K), D?.1 (K), D?.1 (K), J?.3 (Pin_3), R?.2
- net LED_DATA_H: now also J?.2 (Pin_2), Q?.3 (D), R?.2
- net LED_DATA_L: now also Q?.2 (S), R?.2
- net VBUS: now also D?.2 (A), Q?.1, R?.1; no longer C4.1, P_C3.1, P_C4.1, P_L1.2, TVS1.1 (K), U1.3 (VI)
- net VUSB: now also R?.1
- net at UWB_Module1.12 (GPIO3/TXLED): now also R?.1
- net at UWB_Module1.13 (GPIO2/RXLED): now also R?.1
- net at UWB_Module1.14 (GPIO1/SFDLED): now also R?.1
- net at UWB_Module1.15 (GPIO0/RXOKLED): now also R?.1
- new net: C4.1, D?.1 (K), Q?.2, U1.3 (VI)
- new net: D?.2 (A), R?.2 (x4)
- new net +VDC: J?.1 (Pin_1), P_C3.1, P_C4.1, P_L1.2, Q?.3, TVS1.1 (K)
Other:
- moved on the sheet: C1, C16, C18, C2, C3, C4, C5, C6, C7, C8, PS1, P_C1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

Commit message: Finished Schematic Labeling on Hive Bulb PCB v0.2.
Most likely also not going to add more functional components to design.
Parts:
- gave numbers to parts that had none: 14
Changed lines of the file:
@@
 	20250 3850 20250 4250
 $Comp
-L Device:R_US R?
+L Device:R_US R7
 U 1 1 62348BF7
 P 18750 4400
-F 0 "R?" H 18818 4446 50  0000 L CNN
+F 0 "R7" H 18818 4446 50  0000 L CNN
 F 1 "330" H 18818 4355 50  0000 L CNN
 F 2 "Resistor_SMD:R_0805_2012Metric_Pad1.20x1.40mm_HandSolder" V 18790 4390 50  0001 C CNN
@@
 $EndComp
 $Comp
-L Device:R_US R?
+L Device:R_US R8
 U 1 1 6235A7F2
 P 19250 4400
-F 0 "R?" H 19318 4446 50  0000 L CNN
+F 0 "R8" H 19318 4446 50  0000 L CNN
 F 1 "330" H 19318 4355 50  0000 L CNN
 F 2 "Resistor_SMD:R_0805_2012Metric_Pad1.20x1.40mm_HandSolder" V 19290 4390 50  0001 C CNN
@@
 $EndComp
 $Comp
-L Device:R_US R?
+L Device:R_US R9
 U 1 1 6236C4AA
 P 19750 4400
-F 0 "R?" H 19818 4446 50  0000 L CNN
+F 0 "R9" H 19818 4446 50  0000 L CNN
 F 1 "330" H 19818 4355 50  0000 L CNN
 F 2 "Resistor_SMD:R_0805_2012Metric_Pad1.20x1.40mm_HandSolder" V 19790 4390 50  0001 C CNN
@@
 $EndComp
 $Comp
-L Device:R_US R?
+L Device:R_US R10
 U 1 1 6237E261
 P 20250 4400
-F 0 "R?" H 20318 4446 50  0000 L CNN
+F 0 "R10" H 20318 4446 50  0000 L CNN
 F 1 "330" H 20318 4355 50  0000 L CNN
 F 2 "Resistor_SMD:R_0805_2012Metric_Pad1.20x1.40mm_HandSolder" V 20290 4390 50  0001 C CNN
@@
 $EndComp
 $Comp
-L Device:LED D?
-U 1 1 622BAFF3
-P 18750 4850
-F 0 "D?" V 18789 4732 50  0000 R CNN
-F 1 "LED" V 18698 4732 50  0000 R CNN
-F 2 "" H 18750 4850 50  0001 C CNN
-F 3 "~" H 18750 4850 50  0001 C CNN
-	1    18750 4850
-	0    -1   -1   0
-$EndComp
-$Comp
-L Device:LED D?
+L Device:LED RX
 U 1 1 622BAFF4
 P 19250 4850
-F 0 "D?" V 19289 4732 50  0000 R CNN
+F 0 "RX" V 19289 4732 50  0000 R CNN
 F 1 "LED" V 19198 4732 50  0000 R CNN
 F 2 "" H 19250 4850 50  0001 C CNN
@@
 $EndComp
 $Comp
-L Device:LED D?
+L Device:LED SFD
 U 1 1 622BAFF5
 P 19750 4850
-F 0 "D?" V 19789 4732 50  0000 R CNN
+F 0 "SFD" V 19789 4732 50  0000 R CNN
 F 1 "LED" V 19698 4732 50  0000 R CNN
 F 2 "" H 19750 4850 50  0001 C CNN
@@
 $EndComp
 $Comp
-L Device:LED D?
+L Device:LED RXOK
 U 1 1 623A4999
 P 20250 4850
-F 0 "D?" V 20289 4732 50  0000 R CNN
+F 0 "RXOK" V 20289 4732 50  0000 R CNN
 F 1 "LED" V 20198 4732 50  0000 R CNN
 F 2 "" H 20250 4850 50  0001 C CNN
@@
 	19500 5150 19750 5150
 $Comp
-L Connector_Generic:Conn_01x03 J?
+L Connector_Generic:Conn_01x03 J3
 U 1 1 62488C15
 P 18650 7000
-F 0 "J?" H 18568 6675 50  0000 C CNN
+F 0 "J3" H 18568 6675 50  0000 C CNN
 F 1 "Conn_01x03" H 18568 6766 50  0000 C CNN
 F 2 "" H 18650 7000 50  0001 C CNN
@@
 Wire Wire Line
 	18250 7100 18250 7300
-Connection ~ 4800 1750
-Wire Wire Line
-	4800 1750 4800 1850
-$Comp
-L power:GND #PWR0107
-U 1 1 62513991
-P 4800 1850
-F 0 "#PWR0107" H 4800 1600 50  0001 C CNN
-F 1 "GND" H 4805 1677 50  0000 C CNN
-F 2 "" H 4800 1850 50  0001 C CNN
-F 3 "" H 4800 1850 50  0001 C CNN
-	1    4800 1850
-	1    0    0    -1
-$EndComp
-Wire Wire Line
-	4600 1750 4800 1750
-Wire Wire Line
-	4800 1750 5000 1750
 Connection ~ 16750 6450
 Connection ~ 16750 7000
@@
 $EndComp
 $Comp
-L Device:R_US R?
+L Device:R_US R11
 U 1 1 625DBD5D
 P 16750 6650
-F 0 "R?" H 16818 6696 50  0000 L CNN
+F 0 "R11" H 16818 6696 50  0000 L CNN
 F 1 "10K" H 16818 6605 50  0000 L CNN
 F 2 "Resistor_SMD:R_0805_2012Metric_Pad1.20x1.40mm_HandSolder" V 16790 6640 50  0001 C CNN
@@
 $EndComp
 $Comp
-L Device:R_US R?
+L Device:R_US R12
 U 1 1 625DBD63
 P 17750 6650
-F 0 "R?" H 17818 6696 50  0000 L CNN
+F 0 "R12" H 17818 6696 50  0000 L CNN
 F 1 "10K" H 17818 6605 50  0000 L CNN
 F 2 "Resistor_SMD:R_0805_2012Metric_Pad1.20x1.40mm_HandSolder" V 17790 6640 50  0001 C CNN
@@
 $EndComp
 $Comp
-L Transistor_FET:BSS138 Q?
+L Transistor_FET:BSS138 Q2
 U 1 1 625DBD69
 P 17250 6900
-F 0 "Q?" V 17499 6900 50  0000 C CNN
+F 0 "Q2" V 17499 6900 50  0000 C CNN
 F 1 "BSS138" V 17590 6900 50  0000 C CNN
 F 2 "Package_TO_SOT_SMD:SOT-23" H 17450 6825 50  0001 L CIN
@@
 	9350 9150 9350 9250
 $Comp
-L DMG2305UX-7:DMG2305UX-7 Q?
+L DMG2305UX-7:DMG2305UX-7 Q1
 U 1 1 62A55919
 P 4650 11500
-F 0 "Q?" H 4848 11546 50  0000 L CNN
+F 0 "Q1" H 4848 11546 50  0000 L CNN
 F 1 "DMG2305UX-7" H 4848 11455 50  0000 L CNN
 F 2 "SOT91P240X110-3N_DMG2305UX-7" H 4650 11500 50  0001 L BNN
@@
 Connection ~ 4750 11750
 $Comp
-L Device:D_Schottky D?
+L Device:D_Schottky D1
 U 1 1 62B9C55C
 P 4450 11900
-F 0 "D?" H 4450 11683 50  0000 C CNN
+F 0 "D1" H 4450 11683 50  0000 C CNN
 F 1 "D_Schottky" H 4450 11774 50  0000 C CNN
 F 2 "" H 4450 11900 50  0001 C CNN
@@
 	4150 11600 4550 11600
 $Comp
-L Device:R_US R?
+L Device:R_US R11
 U 1 1 62D2F94E
 P 4150 12150
-F 0 "R?" H 4218 12196 50  0000 L CNN
+F 0 "R11" H 4218 12196 50  0000 L CNN
 F 1 "10K" H 4218 12105 50  0000 L CNN
 F 2 "Resistor_SMD:R_0805_2012Metric_Pad1.20x1.40mm_HandSolder" V 4190 12140 50  0001 C CNN
@@
 	16200 2750 16800 2750
 Connection ~ 16800 2750
+$Comp
+L Device:LED TX
+U 1 1 622BAFF3
+P 18750 4850
+F 0 "TX" V 18789 4732 50  0000 R CNN
+F 1 "LED" V 18698 4732 50  0000 R CNN
+F 2 "" H 18750 4850 50  0001 C CNN
+F 3 "~" H 18750 4850 50  0001 C CNN
+	1    18750 4850
+	0    -1   -1   0
+$EndComp
 $EndSCHEMATC
